File: kicad/WordClock.kicad_pcb (KiCad board)
At the start: 2 copper layers, 384.8 x 110.8 mm, 86 parts, among them J1 USB_B_Micro, J10 GND, J2 Conn_01x01, J3 Conn_01x01, J4 DOut, J5 +5V, J6 +5V, J7 +5V, J8 GND, J9 GND, M1 MicrowaveRadarSensorRCWL-0516, Q1 S8050, Q2 S8050, U1 CP2102-GMR_NRND, U2 AMS1117-3.3, U3 ESP-12E

Commit message: PCB routed
Parts:
- J1: footprint barn53_KiCad:MicroUSB_1 -> barn53-kicad:MicroUSB_1
- J10, J4, J5, J6, J7, J8, J9: footprint barn53_KiCad:PCBSolderConnector -> barn53-kicad:PCBSolderConnector; moved to B.Cu
- J2, J3: footprint barn53_KiCad:ThroughHolePin1x1 -> barn53-kicad:ThroughHolePin1x1
- M1: footprint barn53_KiCad:MicrowaveRadarSensorRCWL-0516 -> barn53-kicad:MicrowaveRadarSensorRCWL-0516
- U3: footprint barn53_KiCad:ESP-12E -> barn53-kicad:ESP-12E
- moved J1 2.09 mm to (350.0, 91.8)
- moved CD6 1.20 mm to (245.0, 81.6)
- moved CM1 1.00 mm to (170.6, 118.4)
- moved CM2 1.00 mm to (197.0, 118.4)
- moved CM3 1.00 mm to (223.2, 118.4)
- moved CM4 1.00 mm to (249.5, 118.4)
- moved LEDM1 1.00 mm to (170.6, 113.5)
- moved LEDM2 1.00 mm to (196.9, 113.5)
- moved LEDM3 1.00 mm to (223.1, 113.5)
- moved LEDM4 1.00 mm to (249.4, 113.5)
- moved CD0 0.75 mm to (35.0, 81.6)
- moved CD1 0.75 mm to (70.0, 81.6)
- moved CD10 0.75 mm to (385.0, 81.6)
- moved CD2 0.75 mm to (105.0, 81.6)
- moved CD3 0.75 mm to (140.0, 81.6)
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Routing:
- net VBUS: track 0.00 -> 1701.9 mm, vias 0 -> 50
- net D-: track 0.00 -> 263.1 mm, vias 0 -> 2
- net D+: track 0.00 -> 262.7 mm, vias 0 -> 2
- net Net-(LED0-Pad4): track 0.00 -> 259.9 mm, vias 0 -> 6
- net Move: track 0.00 -> 231.0 mm, vias 0 -> 4
- net +3V3: track 0.00 -> 128.1 mm, vias 0 -> 5
- net Reset: track 0.00 -> 91.4 mm, vias 0 -> 7
- net RxD: track 0.00 -> 91.2 mm, vias 0 -> 7
- net Net-(J2-Pad1): track 0.00 -> 70.2 mm, vias 0 -> 2
- net GND: track 0.00 -> 53.8 mm, vias 0 -> 89
- net GPIO0: track 0.00 -> 48.0 mm, vias 0 -> 2
- net Net-(LED10-Pad2): track 0.00 -> 41.8 mm, vias 0 -> 2
- net TxD: track 0.00 -> 32.2 mm, vias 0 -> 4
- net Net-(LED13-Pad2): track 0.00 -> 31.9 mm
- net Net-(LED12-Pad2): track 0.00 -> 31.9 mm
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Other:
- board size 384.8 x 110.8 mm -> 384.8 x 111.8 mm
- net class Power: trace_width 0.25 -> 0.5
