File: kicad/panel_2_11x10/panel_2_11x10.kicad_pcb (KiCad board)
At the start: 2 copper layers, 384.8 x 76.8 mm, 58 parts, among them J1 DIn, J10 GND, J11 +5V, J12 GND, J13 +5V, J14 GND, J2 +5V, J3 GND, J4 DOut, J5 +5V, J6 +5V, J7 +5V, J8 GND, J9 GND

Commit message: pcb work
Parts:
- moved J11 161.8 mm to (204.5, 93.4)
- moved J12 157.3 mm to (214.6, 93.4)
- moved J2 41.0 mm to (64.5, 93.4)
- moved J14 28.0 mm to (389.6, 93.4)
- moved J3 24.7 mm to (74.4, 93.4)
- moved J1 23.5 mm to (34.5, 93.4)
- moved J13 23.3 mm to (379.5, 93.4)
Routing:
- net VBUS: track 1217.5 -> 1238.8 mm, vias 36 -> 39
- net DIN: track 0.25 -> 20.7 mm, vias 0 -> 1
Other:
- board text added: "WordClock rev.A 11/19"
- board text added: "barn53.de"
